File: CE006_Config feu recompense.kicad_pcb (KiCad board)
At the start: 2 copper layers, 108.7 x 77.1 mm, 81 parts, among them J2 Conn_01x08_Pin, J3 DE9_Socket, J4 DE9_Socket, P1 USB_C_Plug_USB2.0, Q1 FS8205, SW1 SW_SPST, U1 BQ24074RGT, U2 USBLC6-2P6, U3 DW01A, U4 TPS63070RNMR, U5 STM32U073C8Tx, U6 OPA2994xD, U7 ADM3232, Y1 ABM 8.000MHz

Commit message: MAJ PCB + fichiers de fab
Parts:
- added D2: LED ROUGE, LED_SMD:LED_1206_3216Metric, F.Cu at (182.6, 124.1)
- added G***: LOGO, LOGO, B.Cu at (131.3, 123.0)
- D1: value LED_Dual_KKA -> LED VERTE; footprint 5BC-3-CA-F:3_PIN_CONNECTOR -> LED_SMD:LED_1206_3216Metric
- moved D1 2.36 mm to (182.8, 128.3), turned to 0 degrees
Connections:
- D1 pad 1: Net-(D1-K1) -> Net-(D1-K)
- D1 pad 2: Net-(D1-K2) -> Net-(D1-A)
- R5 pad 2: Net-(D1-K2) -> Net-(D1-K)
- R8 pad 2: Net-(D1-K1) -> Net-(D2-K)
Routing:
- net Net-(D1-A): track 113.5 -> 98.1 mm
- net Net-(D1-K2): track 5.25 -> 0.00 mm
- net Net-(D1-K1): track 4.35 -> 0.00 mm
