File: CE006_Config feu recompense.kicad_sch (KiCad schematic)
At the start: 43 parts, among them P1 USB_C_Plug_USB2.0, Q1 FS8205, SW1 SW_SPST, U1 BQ24074RGT, U2 USBLC6-2P6, U3 DW01A, U4 TPS63070RNMR

Commit message: MAJ PCB + fichiers de fab
Parts:
- removed D1: LED_Dual_KKA, 5BC-3-CA-F:3_PIN_CONNECTOR, symbol Device:LED_Dual_KKA
- added D1: LED VERTE, LED_SMD:LED_1206_3216Metric, symbol Device:LED
- added D2: LED ROUGE, LED_SMD:LED_1206_3216Metric, symbol Device:LED
- BT1, TP1, TP2, TP3: now left out of the parts list
Connections:
- net at R8.2: now also D2.1 (K)
- net at R5.2: now also D1.1 (K)
- net at C1.1, SW1.2 (B), U1.10 (OUT)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: now also D1.2 (A), D2.2 (A)
Changed lines of the file:
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@@
 	)
 	(junction
-		(at 260.35 59.69)
-		(diameter 0)
-		(color 0 0 0 0)
-	)
-	(junction
 		(at 220.98 58.42)
 		(diameter 0)
@@
 	)
 	(junction
+		(at 260.35 63.5)
+		(diameter 0)
+		(color 0 0 0 0)
+	)
+	(junction
 		(at 59.69 52.07)
 		(diameter 0)
@@
 	)
 	(junction
+		(at 260.35 55.88)
+		(diameter 0)
+		(color 0 0 0 0)
+	)
+	(junction
 		(at 82.55 127)
 		(diameter 0)
@@
 	(wire
 		(pts
+			(xy 260.35 55.88) (xy 260.35 63.5)
+		)
+		(stroke
+			(width 0)
+			(type default)
+		)
+	)
+	(wire
+		(pts
 			(xy 201.93 130.81) (xy 205.74 130.81)
 		)
@@
 	(wire
 		(pts
+			(xy 251.46 63.5) (xy 260.35 63.5)
+		)
+		(stroke
+			(width 0)
+			(type default)
+		)
+	)
+	(wire
+		(pts
 			(xy 157.48 66.04) (xy 171.45 66.04)
 		)
@@
 	(wire
 		(pts
-			(xy 260.35 74.93) (xy 260.35 59.69)
+			(xy 260.35 38.1) (xy 260.35 55.88)
 		)
 		(stroke
@@
 	(wire
 		(pts
+			(xy 260.35 63.5) (xy 260.35 74.93)
+		)
+		(stroke
+			(width 0)
+			(type default)
+		)
+	)
+	(wire
+		(pts
 			(xy 201.93 107.95) (xy 214.63 107.95)
 		)
@@
 	(wire
 		(pts
-			(xy 241.3 55.88) (xy 241.3 57.15)
+			(xy 149.86 107.95) (xy 149.86 118.11)
 		)
 		(stroke
@@
 	(wire
 		(pts
-			(xy 149.86 107.95) (xy 149.86 118.11)
+			(xy 59.69 52.07) (xy 59.69 54.61)
 		)
 		(stroke
@@
 	(wire
 		(pts
-			(xy 59.69 52.07) (xy 59.69 54.61)
+			(xy 182.88 43.18) (xy 173.99 43.18)
 		)
 		(stroke
@@
 	(wire
 		(pts
-			(xy 182.88 43.18) (xy 173.99 43.18)
+			(xy 179.07 66.04) (xy 195.58 66.04)
 		)
 		(stroke
@@
 	(wire
 		(pts
-			(xy 179.07 66.04) (xy 195.58 66.04)
+			(xy 251.46 55.88) (xy 260.35 55.88)
 		)
 		(stroke
@@
 	(wire
 		(pts
-			(xy 231.14 63.5) (xy 241.3 63.5)
+			(xy 231.14 63.5) (xy 243.84 63.5)
 		)
 		(stroke
@@
 	(wire
 		(pts
-			(xy 231.14 55.88) (xy 241.3 55.88)
+			(xy 231.14 55.88) (xy 243.84 55.88)
 		)
 		(stroke
@@
 	(wire
 		(pts
-			(xy 256.54 59.69) (xy 260.35 59.69)
-		)
-		(stroke
-			(width 0)
-			(type default)
-		)
-	)
-	(wire
-		(pts
 			(xy 264.16 107.95) (xy 261.62 107.95)
 		)
@@
 	(wire
 		(pts
-			(xy 241.3 63.5) (xy 241.3 62.23)
-		)
-		(stroke
-			(width 0)
-			(type default)
-		)
-	)
-	(wire
-		(pts
 			(xy 205.74 133.35) (xy 205.74 135.89)
 		)
@@
 	(wire
 		(pts
-			(xy 260.35 59.69) (xy 260.35 38.1)
-		)
-		(stroke
-			(width 0)
-			(type default)
-		)
-	)
-	(wire
-		(pts
 			(xy 82.55 121.92) (xy 82.55 127)
 		)
@@
 		(body_style 1)
 		(exclude_from_sim no)
-		(in_bom yes)
+		(in_bom no)
 		(on_board yes)
 		(in_pos_files yes)
@@
 	)
 	(symbol
-		(lib_id "Device:LED_Dual_KKA")
-		(at 248.92 59.69 180)
-		(unit 1)
-		(body_style 1)
-		(exclude_from_sim no)
-		(in_bom yes)
-		(on_board yes)
-		(in_pos_files yes)
-		(dnp no)
-		(property "Reference" "D1"
-			(at 248.92 66.04 0)
-			(show_name no)
-			(do_not_autoplace no)
-			(effects
-				(font
-					(size 1.27 1.27)
-				)
-			)
-		)
-		(property "Value" "LED_Dual_KKA"
-			(at 248.92 68.58 0)
-			(show_name no)
-			(do_not_autoplace no)
-			(effects
-				(font
-					(size 1.27 1.27)
-				)
-			)
-		)
-		(property "Footprint" "5BC-3-CA-F:3_PIN_CONNECTOR"
-			(at 247.65 59.69 0)
-			(hide yes)
-			(show_name no)
-			(do_not_autoplace no)
-			(effects
-				(font
-					(size 1.27 1.27)
-				)
-			)
-		)
-		(property "Datasheet" ""
-			(at 247.65 59.69 0)
-			(hide yes)
-			(show_name no)
-			(do_not_autoplace no)
-			(effects
-				(font
-					(size 1.27 1.27)
-				)
-			)
-		)
-		(property "Description" "Dual LED, common anode on pin 3"
-			(at 248.92 59.69 0)
-			(hide yes)
-			(show_name no)
-			(do_not_autoplace no)
-			(effects
-				(font
-					(size 1.27 1.27)
-				)
-			)
-		)
-		(pin "3"
-		)
-		(pin "1"
-		)
-		(pin "2"
-		)
-		(instances
-			(project "CE006_Config feu recompense"
-				(path "/03a83677-8d2d-4975-80a5-1c4b0bd1bc4d"
-					(reference "D1")
-					(unit 1)
-				)
-			)
-		)
-	)
-	(symbol
 		(lib_id "Device:R")
 		(at 177.8 45.72 90)
@@
 		(body_style 1)
 		(exclude_from_sim no)
-		(in_bom yes)
+		(in_bom no)
 		(on_board yes)
 		(in_pos_files yes)
@@
 		(body_style 1)
 		(exclude_from_sim no)
-		(in_bom yes)
+		(in_bom no)
 		(on_board yes)
 		(in_pos_files yes)
@@
 	)
 	(symbol
+		(lib_id "Device:LED")
+		(at 247.65 55.88 0)
+		(unit 1)
+		(body_style 1)
+		(exclude_from_sim no)
+		(in_bom yes)
+		(on_board yes)
+		(in_pos_files yes)
+		(dnp no)
+		(fields_autoplaced yes)
+		(property "Reference" "D1"
+			(at 246.0625 49.53 0)
+			(show_name no)
+			(do_not_autoplace no)
+			(effects
+				(font
+					(size 1.27 1.27)
+				)
+			)
+		)
+		(property "Value" "LED VERTE"
+			(at 246.0625 52.07 0)
+			(show_name no)
+			(do_not_autoplace no)
+			(effects
+				(font
+					(size 1.27 1.27)
+				)
+			)
+		)
+		(property "Footprint" "LED_SMD:LED_1206_3216Metric"
+			(at 247.65 55.88 0)
+			(hide yes)
+			(show_name no)
+			(do_not_autoplace no)
+			(effects
+				(font
+					(size 1.27 1.27)
+				)
+			)
+		)
+		(property "Datasheet" ""
+			(at 247.65 55.88 0)
+			(hide yes)
+			(show_name no)
+			(do_not_autoplace no)
+			(effects
+				(font
+					(size 1.27 1.27)
+				)
+			)
+		)
+		(property "Description" "Light emitting diode"
+			(at 247.65 55.88 0)
+			(hide yes)
+			(show_name no)
+			(do_not_autoplace no)
+			(effects
+				(font
+					(size 1.27 1.27)
+				)
+			)
+		)
+		(property "Sim.Pins" "1=K 2=A"
+			(at 247.65 55.88 0)
+			(hide yes)
+			(show_name no)
+			(do_not_autoplace no)
+			(effects
+				(font
+					(size 1.27 1.27)
+				)
+			)
+		)
+		(pin "1"
+		)
+		(pin "2"
+		)
+		(instances
+			(project "CE006_Config feu recompense"
+				(path "/03a83677-8d2d-4975-80a5-1c4b0bd1bc4d"
+					(reference "D1")
+					(unit 1)
+				)
+			)
+		)
+	)
+	(symbol
 		(lib_id "power:+3.3V")
 		(at 203.2 72.39 0)
@@
 		(body_style 1)
 		(exclude_from_sim no)
-		(in_bom yes)
+		(in_bom no)
 		(on_board yes)
 		(in_pos_files yes)
@@
 					(unit 1)
 				)
+			)
+		)
+	)
+	(symbol
+		(lib_id "Device:LED")
+		(at 247.65 63.5 0)
+		(unit 1)
+		(body_style 1)
+		(exclude_from_sim no)
+		(in_bom yes)
+		(on_board yes)
+		(in_pos_files yes)
+		(dnp no)
+		(property "Reference" "D2"
+			(at 247.142 66.294 0)
+			(show_name no)
+			(do_not_autoplace no)
+			(effects
+				(font
+					(size 1.27 1.27)
+				)
+			)
+		)
+		(property "Value" "LED ROUGE"
+			(at 247.142 68.834 0)
+			(show_name no)
+			(do_not_autoplace no)
+			(effects
+				(font
+					(size 1.27 1.27)
+				)
+			)
+		)
+		(property "Footprint" "LED_SMD:LED_1206_3216Metric"
+			(at 247.65 63.5 0)
+			(hide yes)
+			(show_name no)
+			(do_not_autoplace no)
+			(effects
+				(font
+					(size 1.27 1.27)
+				)
+			)
+		)
+		(property "Datasheet" ""
+			(at 247.65 63.5 0)
+			(hide yes)
+			(show_name no)
+			(do_not_autoplace no)
+			(effects
+				(font
+					(size 1.27 1.27)
+				)
+			)
+		)
+		(property "Description" "Light emitting diode"
+			(at 247.65 63.5 0)
+			(hide yes)
+			(show_name no)
+			(do_not_autoplace no)
+			(effects
+				(font
+					(size 1.27 1.27)
+				)
+			)
+		)
+		(property "Sim.Pins" "1=K 2=A"
+			(at 247.65 63.5 0)
+			(hide yes)
+			(show_name no)
+			(do_not_autoplace no)
+			(effects
+				(font
+					(size 1.27 1.27)
+				)
+			)
+		)
+		(pin "1"
+		)
+		(pin "2"
+		)
+		(instances
+			(project "CE006_Config feu recompense"
+				(path "/03a83677-8d2d-4975-80a5-1c4b0bd1bc4d"
+					(reference "D2")
+					(unit 1)
+				)
