File: MCU.kicad_sch (KiCad schematic)
At the start: 27 parts, among them J1 FTSH-105-01-X-DV-P-K-X, J2 Conn_01x08_Pin, U5 STM32U073C8Tx, U6 OPA2994xD, Y1 ABM 8.000MHz

Commit message: MAJ PCB + fichiers de fab
Parts:
- J1, J2: now left out of the parts list
Changed lines of the file:
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@@
 		(body_style 1)
 		(exclude_from_sim no)
-		(in_bom yes)
+		(in_bom no)
 		(on_board yes)
 		(in_pos_files yes)
@@
 		(body_style 1)
 		(exclude_from_sim no)
-		(in_bom yes)
-		(on_board yes)
-		(in_pos_files yes)
+		(in_bom no)
+		(on_board yes)
+		(in_pos_files yes)
